Commit message: Fixed the Joints to work as expected, It now works as expected with the TelopOpKeyboard Plugin

File: src/threedrover_description/urdf/macros.xacro (robot description, xacro)
@@ -2,42 +2,33 @@
 <robot xmlns:xacro="https://www.ros.org/wiki/xacro">
 <!-- LINK_BOGIE ********************************************************** -->
-	<macro name ="link_bogie_stat" params="name orientation">
+	<macro name ="link_bogie_stat" params="name">
 		<link name="${name}">
 			<!-- values from the fusion360 files -->
 		    <inertial>
 		      <mass value="0.2"/>
-		      <origin rpy="${1.570796*orientation} 0 0" xyz="0 ${-0.15516*orientation} 0"/>
 		      <inertia ixx="0.000526666666667" ixy="0" ixz="0" iyy="0.000526666666667" iyz="0" izz="0.001"/>
 		    </inertial>
 		    <collision name="${name}_collision">
-		      <origin rpy="${1.570796*orientation} 0 0" xyz="0 ${-0.15516*orientation} 0"/>
 	      		<geometry>
-				<mesh filename="package://threedrover_description/MODELS/OWR_20_BOGIE_00_ASM_STAT.stl" scale="0.001 0.001 0.001" />
+				<cylinder length="0.05" radius="0.05"/>
+				<!--<mesh filename="package://threedrover_description/MODELS/OWR_20_BOGIE_00_ASM_STAT.stl" scale="0.001 0.001 0.001" />-->
   		        </geometry>
 		    </collision>
 		    <visual name="${name}_visual">
-		      <origin rpy="${1.570796*orientation} 0 0" xyz="0 ${-0.15516*orientation} 0"/>
 		      	<geometry>
-				<mesh filename="package://threedrover_description/MODELS/OWR_20_BOGIE_00_ASM_STAT.stl" scale="0.001 0.001 0.001" />
+				<cylinder length="0.05" radius="0.05"/>
+				<!--<mesh filename="package://threedrover_description/MODELS/OWR_20_BOGIE_00_ASM_STAT.stl" scale="0.001 0.001 0.001" />-->
 		     	 </geometry>
 		    </visual>
 	   	</link>
     	</macro>
-	<macro name ="link_bogie_rot" params="name orientation">
+	<macro name ="link_bogie_rot" params="name">
 		<link name="${name}">
 			<!-- values from the fusion360 files -->
 		    <inertial>
 		      <mass value="0.2"/>
-		      <origin rpy="${1.570796*orientation} ${(orientation ==-1)*(3.14) +orientation*0.06925171} 0" xyz="0 ${-0.15516*orientation} 0"/>
 		      <inertia ixx="0.000526666666667" ixy="0" ixz="0" iyy="0.000526666666667" iyz="0" izz="0.001"/>
 		    </inertial>
-		    <collision name="${name}_collision">
-		      <origin rpy="${1.570796*orientation} ${(orientation ==-1)*3.14 +orientation*0.06925171} 0" xyz="0 ${-0.15516*orientation} 0"/>
-	      		<geometry>
-				<mesh filename="package://threedrover_description/MODELS/OWR_20_BOGIE_00_ASM_ROT.stl" scale="0.001 0.001 0.001" />
-  		        </geometry>
-		    </collision>
 		    <visual name="${name}_visual">
-		      <origin rpy="${1.570796*orientation} ${(orientation ==-1)*3.14 +orientation*0.06925171} 0" xyz="0 ${-0.15516*orientation} 0"/>
 		      	<geometry>
 				<mesh filename="package://threedrover_description/MODELS/OWR_20_BOGIE_00_ASM_ROT.stl" scale="0.001 0.001 0.001" />
@@ -52,39 +43,36 @@
 		    <inertial>
 		      <mass value="0.2"/>
-		      <origin rpy="${1.570796*orientation} 0 0" xyz="${-0.3865*end} ${-(0.15516+0.134 + 0.078)*orientation} -0.22012"/>
 		      <inertia ixx="0.000526666666667" ixy="0" ixz="0" iyy="0.000526666666667" iyz="0" izz="0.001"/>
 		    </inertial>
 		    <collision name="${name}_collision">
-		      <origin rpy="${1.570796*orientation} 0 0" xyz="${-0.3865*end} ${-(0.15516+0.134 + 0.078)*orientation} -0.22012"/>
 	      		<geometry>
-				<mesh filename="package://threedrover_description/MODELS/OWR_20_DRIVE_00_ASM_STAT.stl" scale="0.001 0.001 0.001" />
+				<cylinder length="0.05" radius="0.05"/>
   		        </geometry>
 		    </collision>
 		    <visual name="${name}_visual">
-		      <origin rpy="${1.570796*orientation} 0 0" xyz="${-0.3865*end} ${-(0.15516+0.134 + 0.078)*orientation} -0.22012"/>
 		      	<geometry>
-				<mesh filename="package://threedrover_description/MODELS/OWR_20_DRIVE_00_ASM_STAT.stl" scale="0.001 0.001 0.001" />
+				<cylinder length="0.05" radius="0.05"/>
+				<!-- <mesh filename="package://threedrover_description/MODELS/OWR_20_DRIVE_00_ASM_STAT.stl" scale="0.001 0.001 0.001" /> -->
 		     	 </geometry>
 		    </visual>
 	   	</link>
     	</macro>
-	<macro name ="link_wheel_rot" params="name orientation end">
+	<macro name ="link_wheel_rot" params="name  orientation end">
 		<link name="${name}">
 			<!-- values from the fusion360 files -->
 		    <inertial>
 		      <mass value="0.2"/>
-		      <origin rpy="${1.570796*orientation} ${(orientation ==-1)*3.14} 0" xyz="${-0.3865*end} ${-(0.15516+0.134 + 0.078)*orientation} -0.22012"/>
 		      <inertia ixx="0.000526666666667" ixy="0" ixz="0" iyy="0.000526666666667" iyz="0" izz="0.001"/>
 		    </inertial>
 		    <collision name="${name}_collision">
-		      <origin rpy="${1.570796*orientation} ${(orientation ==-1)*3.14} 0" xyz="${-0.3865*end} ${-(0.15516+0.134 + 0.078)*orientation} -0.22012"/>
-	      		<geometry>
-				<mesh filename="package://threedrover_description/MODELS/OWR_20_DRIVE_00_ASM_ROT.stl" scale="0.001 0.001 0.001" />
-  		        </geometry>
+				<geometry>
+			<!--	<mesh filename="package://threedrover_description/MODELS/OWR_20_DRIVE_00_ASM_ROT.stl" scale="0.001 0.001 0.001" /> -->
+				<cylinder length="0.098" radius="0.1"/>
+			</geometry>
 		    </collision>
 		    <visual name="${name}_visual">
-		      <origin rpy="${1.570796*orientation} ${(orientation ==-1)*3.14} 0" xyz="${-0.3865*end} ${-(0.15516+0.134 + 0.078)*orientation} -0.22012"/>
 		      	<geometry>
-				<mesh filename="package://threedrover_description/MODELS/OWR_20_DRIVE_00_ASM_ROT.stl" scale="0.001 0.001 0.001" />
+				<!--	<mesh filename="package://threedrover_description/MODELS/OWR_20_DRIVE_00_ASM_ROT.stl" scale="0.001 0.001 0.001" /> -->
+				<cylinder length="0.098" radius="0.1"/>
 		     	 </geometry>
 		    </visual>
@@ -92,9 +80,10 @@
     	</macro>
 <!-- JOINTS ********************************************************** -->
-	<macro name="joint_stat" params="name child parent origin_xyz" >
+	<macro name="joint_bogie_stat" params="name child parent orientation" >
     		<joint name="${name}" type="fixed">
-			<origin rpy="0 0 0" xyz="${origin_xyz}"/>
+		      <!-- <origin rpy="${1.570796*orientation} 0 0" xyz="0 ${-0.15516*orientation} 0"/> -->
+		      <origin rpy="${1.570796*orientation} 0 0" xyz="0 ${-0.15516*orientation} 0"/>
 			<child link="${child}"/>
-			<parent link="link_chassis"/>
+			<parent link="${parent}"/>
 			<axis rpy="1.570796 0 0" xyz="0 1 0"/>
 			<limit effort="10000" velocity="1000"/>
@@ -102,10 +91,37 @@
 		</joint>
     	</macro>
-	<macro name="joint_rot" params="name child parent origin_xyz" >
+	<macro name="joint_bogie_rot" params="name child parent orientation" >
     		<joint name="${name}" type="continuous">
-			<origin rpy="0 0 0" xyz="${origin_xyz}"/>
+		     <!-- <origin rpy="0 ${(orientation ==-1)*3.14 + orientation*0.06925171} 0" xyz="0 0 0"/> -->
+			<origin rpy="0 0 ${(orientation ==-1)*3.14 + orientation*0.06925171}" xyz="0 0 0"/>
 			<child link="${child}"/>
 			<parent link="${parent}"/>
-			<axis rpy="0 0 0" xyz="0 1 0"/>
+			<axis rpy="0 0 0" xyz="0 0 1"/>
+			<limit effort="10000" velocity="1000"/>
+			<joint_properties damping="1.0" friction="1.0"/>
+		</joint>
+    	</macro>
+<!--WHEEL JOINTS ********************************************************** -->
+	<macro name="wheel_joint_stat" params="name child parent orientation end" >
+    		<joint name="${name}" type="fixed">
+			<!-- one leg goes (0.4006 and -0.193183) while the other goes (-0.370 and -0.247057)  using vector magic the
+				wheel positions can be paramaterised for end =1 or end = -1 -->
+			<origin rpy="0 0 ${1.570796*orientation}" xyz="${0.0153 + 0.3853*end} ${-0.22012 + 0.026937*end} 0.17"/>
+			<child link="${child}"/>
+			<parent link="${parent}"/>
+			<axis rpy="1.570796 0 0" xyz="0 0 1"/>
+			<limit effort="10000" velocity="1000"/>
+			<joint_properties damping="1.0" friction="1.0"/>
+		</joint>
+    	</macro>
+	<macro name="wheel_joint_rot" params="name child parent orientation end" >
+    		<joint name="${name}" type="continuous">
+			<!--<origin rpy="0 0 0" xyz="${-0.3865*end} ${-(0.15516+0.134 + 0.078)*orientation} -0.22012"/> -->
+			<!--
+			<origin rpy="${1.570796*orientation} ${(orientation ==-1)*3.14} 0" xyz="${-0.3865*end} ${-(0.15516+0.134 + 0.078)*orientation} -0.22012"/> -->
+			<origin rpy="0 0 0" xyz="0 0 0.05"/>
+			<child link="${child}"/>
+			<parent link="${parent}"/>
+			<axis rpy="0 0 0" xyz="0 0 1"/>
 			<limit effort="10000" velocity="1000"/>
 			<joint_properties damping="1.0" friction="1.0"/>

File: src/threedrover_description/urdf/rover.xacro (robot description, xacro)
@@ -3,8 +3,9 @@
 	<xacro:include filename="macros.xacro" />
 	<xacro:include filename="mats.xacro" />
+	<xacro:include filename="rover.gazebo"/>
 	<link name="link_chassis">
 		<!-- values calculated in fusion360 -->
 		<inertial>
-			<mass value="10"/>
+			<mass value="2.441483"/>
 			<origin rpy="0 0 0" xyz="0 0 0"/>
 			<inertia
@@ -33,29 +34,28 @@
 	</link>
 	<!-- Bogie -->
-	<xacro:link_bogie_stat name="link_right_bogie_stat"  orientation="1" />
-	<xacro:link_bogie_rot name="link_right_bogie_rot"  orientation="1"/>
-	<xacro:link_bogie_stat name="link_left_bogie_stat" orientation="-1"/>
-	<xacro:link_bogie_rot name="link_left_bogie_rot" orientation="-1" />
-g
-	<xacro:joint_stat name="joint_bogie_left_stat" child="link_left_bogie_stat" parent="joint_chassis" origin_xyz="0 0 0"/>
-	<xacro:joint_stat name="joint_bogie_right_stat" child="link_right_bogie_stat" parent="joint_chassis" origin_xyz="0 0 0"/>
-	<xacro:joint_rot name="joint_bogie_right_rot" child="link_right_bogie_rot" parent="link_right_bogie_stat" origin_xyz="0 0 0"/>
-	<xacro:joint_rot name="joint_bogie_left_rot" child="link_left_bogie_rot" parent="link_left_bogie_stat" origin_xyz="0 0 0"/>
+	<xacro:link_bogie_stat name="link_right_bogie_stat" />
+	<xacro:link_bogie_rot name="link_right_bogie_rot"/>
+	<xacro:link_bogie_stat name="link_left_bogie_stat" />
+	<xacro:link_bogie_rot name="link_left_bogie_rot"/>
+	<xacro:joint_bogie_stat name="joint_bogie_left_stat" child="link_left_bogie_stat" parent="link_chassis"   orientation="-1"/>
+	<xacro:joint_bogie_stat name="joint_bogie_right_stat" child="link_right_bogie_stat" parent="link_chassis"  orientation="1"/>
+	<xacro:joint_bogie_rot name="joint_bogie_right_rot" child="link_right_bogie_rot" parent="link_right_bogie_stat"  orientation="1"/>
+	<xacro:joint_bogie_rot name="joint_bogie_left_rot" child="link_left_bogie_rot" parent="link_left_bogie_stat" orientation="-1"/>
 	<!-- Wheel -->
 	<xacro:link_wheel_stat name="link_FRSWheel"  orientation="1" end="1"/>
+	<xacro:link_wheel_stat name="link_FLSWheel"  orientation="-1" end="1"/>
 	<xacro:link_wheel_stat name="link_BRSWheel"  orientation="1" end="-1"/>
-	<xacro:link_wheel_stat name="link_FLSWheel"  orientation="-1" end="1"/>
 	<xacro:link_wheel_stat name="link_BLSWheel"  orientation="-1" end="-1"/>
+	<xacro:wheel_joint_stat name="wheelmount_FL" child="link_FLSWheel" parent="link_left_bogie_rot" orientation="-1" end="-1"/>
+	<xacro:wheel_joint_stat name="wheelmount_BL" child="link_BLSWheel" parent="link_left_bogie_rot" orientation="-1" end="1"/>
+	<xacro:wheel_joint_stat name="wheelmount_FR" child="link_FRSWheel" parent="link_right_bogie_rot" orientation="1" end="1"/>
+	<xacro:wheel_joint_stat name="wheelmount_BR" child="link_BRSWheel" parent="link_right_bogie_rot" orientation="1" end="-1"/>
 	<xacro:link_wheel_rot name="link_FRRWheel"  orientation="1" end="1"/>
 	<xacro:link_wheel_rot name="link_BRRWheel"  orientation="1" end="-1"/>
 	<xacro:link_wheel_rot name="link_FLRWheel"  orientation="-1" end="1"/>
 	<xacro:link_wheel_rot name="link_BLRWheel"  orientation="-1" end="-1"/>
-	<xacro:joint_stat name="wheelmount_FL" child="link_FLSWheel" parent="link_left_bogie_rot" origin_xyz="0 0 0"/>
-	<xacro:joint_stat name="wheelmount_BL" child="link_BLSWheel" parent="link_left_bogie_rot" origin_xyz="0 0 0"/>
-	<xacro:joint_stat name="wheelmount_FR" child="link_FRSWheel" parent="link_right_bogie_rot" origin_xyz="0 0 0"/>
-	<xacro:joint_stat name="wheelmount_BR" child="link_BRSWheel" parent="link_right_bogie_rot" origin_xyz="0 0 0"/>
-	<xacro:joint_stat name="wheel_FL" child="link_FLRWheel" parent="link_FLSWheel" origin_xyz="0 0 0"/>
-	<xacro:joint_stat name="wheel_BL" child="link_BLRWheel" parent="link_BLSWheel" origin_xyz="0 0 0"/>
-	<xacro:joint_stat name="wheel_FR" child="link_FRRWheel" parent="link_FRSWheel" origin_xyz="0 0 0"/>
-	<xacro:joint_stat name="wheel_BR" child="link_BRRWheel" parent="link_BRSWheel" origin_xyz="0 0 0"/>
+	<xacro:wheel_joint_rot name="wheel_FL" child="link_FLRWheel" parent="link_FLSWheel" orientation="-1" end="1"/>
+	<xacro:wheel_joint_rot name="wheel_BL" child="link_BLRWheel" parent="link_BLSWheel" orientation="-1" end="-1"/>
+	<xacro:wheel_joint_rot name="wheel_FR" child="link_FRRWheel" parent="link_FRSWheel" orientation="1" end="1"/>
+	<xacro:wheel_joint_rot name="wheel_BR" child="link_BRRWheel" parent="link_BRSWheel" orientation="1" end="-1"/>
 </robot>

Commit message: inertia added

File: src/threedrover_description/urdf/macros.xacro (robot description, xacro)
@@ -5,8 +5,20 @@
 		<link name="${name}">
 			<!-- values from the fusion360 files -->
-		    <inertial>
-		      <mass value="0.2"/>
+		<inertial>
+			<mass value="0.441"/>
+			<origin rpy="0 0 0" xyz="-0.00000069097  0.0002123 0.038"/>
+			<inertia
+				ixx =  "0.002"
+				ixy =  "-0.00003576"
+				ixz =  "-0.000000003393"
+				iyy =  "0.000779"
+				iyz =  "0.00000003725"
+				izz =  "0.002"
+			/>
+		</inertial>
+		  <!--  <inertial>
+		      <mass value="0.441"/>
 		      <inertia ixx="0.000526666666667" ixy="0" ixz="0" iyy="0.000526666666667" iyz="0" izz="0.001"/>
-		    </inertial>
+		    </inertial> -->
 		    <collision name="${name}_collision">
 	      		<geometry>
@@ -26,8 +38,9 @@
 		<link name="${name}">
 			<!-- values from the fusion360 files -->
-		    <inertial>
-		      <mass value="0.2"/>
-		      <inertia ixx="0.000526666666667" ixy="0" ixz="0" iyy="0.000526666666667" iyz="0" izz="0.001"/>
-		    </inertial>
+		<inertial>
+			<mass value="0.871251"/>
+			<origin rpy="0 0 0" xyz="0.004  -0.077 0.091"/>
+			<inertia ixx =  "0.009" ixy =  "-0.002" ixz =  "${-9.081*0.00001}" iyy =  "0.039" iyz =  "0.002" izz =  "0.045" />
+		</inertial>
 		    <visual name="${name}_visual">
 		      	<geometry>
@@ -41,8 +54,9 @@
 		<link name="${name}">
 			<!-- values from the fusion360 files -->
-		    <inertial>
-		      <mass value="0.2"/>
-		      <inertia ixx="0.000526666666667" ixy="0" ixz="0" iyy="0.000526666666667" iyz="0" izz="0.001"/>
-		    </inertial>
+			<inertial>
+				<mass value="1.397"/>
+				<origin rpy="0 0 0" xyz="0.003  -0.003 0.013"/>
+				<inertia ixx =  "0.002" ixy =  "-0.000006590" ixz =  "0.0001390" iyy =  "0.002" iyz =  "-0.0000004779" izz =  "0.002" />
+			</inertial>
 		    <collision name="${name}_collision">
 	      		<geometry>
@@ -61,8 +75,9 @@
 		<link name="${name}">
 			<!-- values from the fusion360 files -->
-		    <inertial>
-		      <mass value="0.2"/>
-		      <inertia ixx="0.000526666666667" ixy="0" ixz="0" iyy="0.000526666666667" iyz="0" izz="0.001"/>
-		    </inertial>
+			<inertial>
+				<mass value="6.598"/>
+				<origin rpy="0 0 0" xyz="-0.003  -0.003 0.026"/>
+				<inertia ixx =  "0.031" ixy =  "0.0000002489" ixz =  "-0.000000001240" iyy =  "0.031" iyz =  "0.00000001531" izz =  "0.051" />
+			</inertial>
 		    <collision name="${name}_collision">
 				<geometry>

File: src/threedrover_description/urdf/rover.xacro (robot description, xacro)
@@ -8,12 +8,12 @@
 		<inertial>
 			<mass value="2.441483"/>
-			<origin rpy="0 0 0" xyz="0 0 0"/>
+			<origin rpy="0 0 0" xyz="0  0 0"/>
 			<inertia
-				ixx =  "0.06062"
-				ixy =  "0.0003601"
-				ixz = "-0.00002478"
-				iyy =  "0.0003601"
-				iyz =  "0"
-				izz =  "0.08117"
+				ixx =  "0.061"
+				ixy =  "${3.601*0.0001}"
+				ixz =  "${-2.478*0.00001}"
+				iyy =  "${0.119}"
+				iyz =  "${5.191*0.0000001}"
+				izz =  "${0.081}"
 			/>
 		</inertial>

Commit message: added camera and lidar sensors, as well as replacing stl mesh with prism for performance reasons

File: src/threedrover_description/urdf/macros.xacro (robot description, xacro)
@@ -95,4 +95,15 @@
     	</macro>
 <!-- JOINTS ********************************************************** -->
+	<macro name="joint_sensor" params="name child parent pos" >
+    		<joint name="${name}" type="fixed">
+		      <!-- <origin rpy="${1.570796*orientation} 0 0" xyz="0 ${-0.15516*orientation} 0"/> -->
+		      <origin rpy="0 0 0" xyz="${pos}"/>
+			<child link="${child}"/>
+			<parent link="${parent}"/>
+			<axis rpy="1.570796 0 0" xyz="0 1 0"/>
+			<limit effort="10000" velocity="1000"/>
+			<joint_properties damping="1.0" friction="1.0"/>
+		</joint>
+    	</macro>
 	<macro name="joint_bogie_stat" params="name child parent orientation" >
     		<joint name="${name}" type="fixed">

File: src/threedrover_description/urdf/rover.xacro (robot description, xacro)
@@ -27,5 +27,6 @@
 		<visual>
 			<geometry>
-				<mesh filename="package://threedrover_description/MODELS/OWR_20_CHASSIS_00_ASM.stl" scale="0.001 0.001 0.001" />
+				<!--<mesh filename="package://threedrover_description/MODELS/OWR_20_CHASSIS_00_ASM.stl" scale="0.001 0.001 0.001" />-->
+				<box size = "0.511 0.208 0.4"/>
 			</geometry>
 			<origin rpy="1.570796 0 0" xyz="0 0 0"/>
@@ -59,3 +60,23 @@
 	<xacro:wheel_joint_rot name="wheel_FR" child="link_FRRWheel" parent="link_FRSWheel" orientation="1" end="1"/>
 	<xacro:wheel_joint_rot name="wheel_BR" child="link_BRRWheel" parent="link_BRSWheel" orientation="1" end="-1"/>
+	<link name = "camera_link">
+		<visual>
+			<geometry>
+				<box size="0.1 0.1 0.1"/>
+			</geometry>
+		</visual>
+			<origin rpy="0 0 0" xyz="0 0 0"/>
+     			<material name="green"/>
+	</link>
+	<link name = "lidar_link">
+		<visual>
+			<geometry>
+				<box size="0.05 0.05 0.1"/>
+			</geometry>
+		</visual>
+			<origin rpy="0 0 0" xyz="0 0 0"/>
+     			<material name="green"/>
+	</link>
+	<xacro:joint_sensor name="camera_joint" child="camera_link" parent="link_chassis" pos="0.2555 0 0"/>
+	<xacro:joint_sensor name="lidar_joint" child="lidar_link" parent="link_chassis" pos="0.2275 0 0.104"/>
 </robot>

Commit message: fixed differential to work correctly by connecting both bogies to the same rotational joint

File: src/threedrover_description/urdf/macros.xacro (robot description, xacro)
@@ -117,8 +117,19 @@
 		</joint>
     	</macro>
+	<macro name="joint_bogie_stat2" params="name child parent orientation" >
+    		<joint name="${name}" type="fixed">
+		      <!-- <origin rpy="${1.570796*orientation} 0 0" xyz="0 ${-0.15516*orientation} 0"/> -->
+		      <origin rpy="0 3.14159 0.11" xyz="0 0 ${-2*0.15516}"/>
+			<child link="${child}"/>
+			<parent link="${parent}"/>
+			<axis rpy="1.570796 0 0" xyz="0 1 0"/>
+			<limit effort="10000" velocity="1000"/>
+			<joint_properties damping="1.0" friction="1.0"/>
+		</joint>
+    	</macro>
 	<macro name="joint_bogie_rot" params="name child parent orientation" >
     		<joint name="${name}" type="continuous">
 		     <!-- <origin rpy="0 ${(orientation ==-1)*3.14 + orientation*0.06925171} 0" xyz="0 0 0"/> -->
-			<origin rpy="0 0 ${(orientation ==-1)*3.14 + orientation*0.06925171}" xyz="0 0 0"/>
+			<origin rpy="0 0 ${(orientation ==-1)*3.14159}" xyz="0 0 0"/>
 			<child link="${child}"/>
 			<parent link="${parent}"/>

File: src/threedrover_description/urdf/rover.xacro (robot description, xacro)
@@ -42,5 +42,5 @@
 	<xacro:joint_bogie_stat name="joint_bogie_right_stat" child="link_right_bogie_stat" parent="link_chassis"  orientation="1"/>
 	<xacro:joint_bogie_rot name="joint_bogie_right_rot" child="link_right_bogie_rot" parent="link_right_bogie_stat"  orientation="1"/>
-	<xacro:joint_bogie_rot name="joint_bogie_left_rot" child="link_left_bogie_rot" parent="link_left_bogie_stat" orientation="-1"/>
+	<xacro:joint_bogie_stat2 name="joint_bogie_left_rot" child="link_left_bogie_rot" parent="link_right_bogie_rot" orientation="-1"/>
 	<!-- Wheel -->
 	<xacro:link_wheel_stat name="link_FRSWheel"  orientation="1" end="1"/>

Commit message: added teleoptwist for testing purposes, differential is now completely open

File: src/threedrover_description/urdf/macros.xacro (robot description, xacro)
@@ -88,6 +88,6 @@
 		    <visual name="${name}_visual">
 		      	<geometry>
-				<!--	<mesh filename="package://threedrover_description/MODELS/OWR_20_DRIVE_00_ASM_ROT.stl" scale="0.001 0.001 0.001" /> -->
-				<cylinder length="0.098" radius="0.1"/>
+					<mesh filename="package://threedrover_description/MODELS/OWR_20_DRIVE_00_ASM_ROT.stl" scale="0.001 0.001 0.001" />
+				<!--<cylinder length="0.098" radius="0.1"/> -->
 		     	 </geometry>
 		    </visual>
@@ -117,13 +117,14 @@
 		</joint>
     	</macro>
-	<macro name="joint_bogie_stat2" params="name child parent orientation" >
-    		<joint name="${name}" type="fixed">
-		      <!-- <origin rpy="${1.570796*orientation} 0 0" xyz="0 ${-0.15516*orientation} 0"/> -->
-		      <origin rpy="0 3.14159 0.11" xyz="0 0 ${-2*0.15516}"/>
+	<macro name="joint_bogie_rot2" params="name child parent orientation mimic" >
+    		<joint name="${name}" type="continuous">
+		      <!-- <origin rpy="${1.570796*orientation} 0 ${0.26937/2}" xyz="0 ${-0.15516*orientation} 0"/> -->
+		      <origin rpy="0 0 ${(orientation ==-1)*3.14159}" xyz="0 0 0"/>
 			<child link="${child}"/>
 			<parent link="${parent}"/>
-			<axis rpy="1.570796 0 0" xyz="0 1 0"/>
+			<axis rpy="1.570796 0 0" xyz="0 0 1"/>
 			<limit effort="10000" velocity="1000"/>
 			<joint_properties damping="1.0" friction="1.0"/>
+			<mimic joint="${mimic}" multiplier="-1" offset="0"/>
 		</joint>
     	</macro>
@@ -157,5 +158,5 @@
 			<!--
 			<origin rpy="${1.570796*orientation} ${(orientation ==-1)*3.14} 0" xyz="${-0.3865*end} ${-(0.15516+0.134 + 0.078)*orientation} -0.22012"/> -->
-			<origin rpy="0 0 0" xyz="0 0 0.05"/>
+			<origin rpy="0 0 ${1.570796*orientation}" xyz="0 0 0.05"/>
 			<child link="${child}"/>
 			<parent link="${parent}"/>

File: src/threedrover_description/urdf/rover.xacro (robot description, xacro)
@@ -34,4 +34,6 @@
 		</visual>
 	</link>
+	<!-- Differential -->
+		<!-- Diif bar -->
 	<!-- Bogie -->
 	<xacro:link_bogie_stat name="link_right_bogie_stat" />
@@ -42,5 +44,5 @@
 	<xacro:joint_bogie_stat name="joint_bogie_right_stat" child="link_right_bogie_stat" parent="link_chassis"  orientation="1"/>
 	<xacro:joint_bogie_rot name="joint_bogie_right_rot" child="link_right_bogie_rot" parent="link_right_bogie_stat"  orientation="1"/>
-	<xacro:joint_bogie_stat2 name="joint_bogie_left_rot" child="link_left_bogie_rot" parent="link_right_bogie_rot" orientation="-1"/>
+	<xacro:joint_bogie_rot name="joint_bogie_left_rot" child="link_left_bogie_rot" parent="link_left_bogie_stat" orientation="-1"/>
 	<!-- Wheel -->
 	<xacro:link_wheel_stat name="link_FRSWheel"  orientation="1" end="1"/>
