Commit message: turning works now thank fuck

File: src/threedrover_description/urdf/macros.xacro (robot description, xacro)
@@ -81,12 +81,23 @@
 			</inertial>
 		    <collision name="${name}_collision">
+				<origin rpy="0 0 0" xyz="0  0 0"/>
 				<geometry>
-			<!--	<mesh filename="package://threedrover_description/MODELS/OWR_20_DRIVE_00_ASM_ROT.stl" scale="0.001 0.001 0.001" /> -->
+			<!--	<mesh filename="package://threedrover_description/MODELS/OWR_20_DRIVE_00_ASM_ROT.stl" scale="0.001 0.001 0.001" /> ${3.14159*orientation*(-1)}-->
 				<cylinder length="0.098" radius="0.1"/>
 			</geometry>
+			<friction>
+				<ode>
+					<mu> 2 </mu>
+					<mu2> 1.8 </mu2>
+				</ode>
+			</friction>
+			<contact>
+				<min_depth>0.01</min_depth>
+			</contact>
 		    </collision>
 		    <visual name="${name}_visual">
+				<origin rpy="${3.14159*orientation*(-1)} 0 0" xyz="0  0 0.026"/>
 		      	<geometry>
-					<mesh filename="package://threedrover_description/MODELS/OWR_20_DRIVE_00_ASM_ROT.stl" scale="0.001 0.001 0.001" />
+				<mesh filename="package://threedrover_description/MODELS/OWR_20_DRIVE_00_ASM_ROT.stl" scale="0.001 0.001 0.001" />
 				<!--<cylinder length="0.098" radius="0.1"/> -->
 		     	 </geometry>
@@ -119,5 +130,5 @@
 	<macro name="joint_bogie_rot2" params="name child parent orientation mimic" >
     		<joint name="${name}" type="continuous">
-		      <!-- <origin rpy="${1.570796*orientation} 0 ${0.26937/2}" xyz="0 ${-0.15516*orientation} 0"/> -->
+		      <!-- <origin rpy="${1.570796*orientation} 0 ${0.26937/2}" xyz="0 ${-0.15516*orientation} 0"/>${(orientation ==-1)*3.14159} -->
 		      <origin rpy="0 0 ${(orientation ==-1)*3.14159}" xyz="0 0 0"/>
 			<child link="${child}"/>
@@ -131,5 +142,5 @@
 	<macro name="joint_bogie_rot" params="name child parent orientation" >
     		<joint name="${name}" type="continuous">
-		     <!-- <origin rpy="0 ${(orientation ==-1)*3.14 + orientation*0.06925171} 0" xyz="0 0 0"/> -->
+		     <!-- <origin rpy="0 ${(orientation ==-1)*3.14 + orientation*0.06925171} 0" xyz="0 0 0"/> ${(orientation ==-1)*3.14159}-->
 			<origin rpy="0 0 ${(orientation ==-1)*3.14159}" xyz="0 0 0"/>
 			<child link="${child}"/>
@@ -137,5 +148,5 @@
 			<axis rpy="0 0 0" xyz="0 0 1"/>
 			<limit effort="10000" velocity="1000"/>
-			<joint_properties damping="1.0" friction="1.0"/>
+			<joint_properties damping="10.0" friction="100.0"/>
 		</joint>
     	</macro>
@@ -145,5 +156,5 @@
 			<!-- one leg goes (0.4006 and -0.193183) while the other goes (-0.370 and -0.247057)  using vector magic the
 				wheel positions can be paramaterised for end =1 or end = -1 -->
-			<origin rpy="0 0 ${1.570796*orientation}" xyz="${0.0153 + 0.3853*end} ${-0.22012 + 0.026937*end} 0.17"/>
+			<origin rpy="${(orientation ==1)*3.14159} 0 ${1.570796*orientation}" xyz="${0.0153 + 0.3853*end} ${-0.22012 + 0.026937*end} 0.17"/>
 			<child link="${child}"/>
 			<parent link="${parent}"/>
@@ -158,5 +169,5 @@
 			<!--
 			<origin rpy="${1.570796*orientation} ${(orientation ==-1)*3.14} 0" xyz="${-0.3865*end} ${-(0.15516+0.134 + 0.078)*orientation} -0.22012"/> -->
-			<origin rpy="0 0 ${1.570796*orientation}" xyz="0 0 0.05"/>
+			<origin rpy="0 0 ${1.570796*orientation}" xyz="0 0 ${0.05*orientation*(-1)}"/>
 			<child link="${child}"/>
 			<parent link="${parent}"/>

File: src/threedrover_description/urdf/rover.xacro (robot description, xacro)
@@ -19,9 +19,9 @@
 		</inertial>
 		<collision>
+			<origin rpy="0 0 0" xyz="0 0 0"/>
 			<geometry>
 				<!--Again this is from the fusion360-->
 				<box size = "0.511 0.4 0.208"/>
 			</geometry>
-			<origin rpy="1.570796 0 0" xyz="0 0 0"/>
 		</collision>
 		<visual>

Commit message: added topics to control joint velocities directly

File: src/threedrover_description/urdf/macros.xacro (robot description, xacro)
@@ -88,10 +88,10 @@
 			<friction>
 				<ode>
-					<mu> 2 </mu>
-					<mu2> 1.8 </mu2>
+					<mu> 0.9 </mu>
+					<mu2> 0.8 </mu2>
 				</ode>
 			</friction>
 			<contact>
-				<min_depth>0.01</min_depth>
+				<min_depth>0.001</min_depth>
 			</contact>
 		    </collision>
@@ -173,7 +173,21 @@
 			<parent link="${parent}"/>
 			<axis rpy="0 0 0" xyz="0 0 1"/>
-			<limit effort="10000" velocity="1000"/>
-			<joint_properties damping="1.0" friction="1.0"/>
+			<limit
+			lower="0"
+			upper="3.14"
+			effort="2"
+			velocity="2.0" />
+			<joint_properties damping="1.0" friction="0.2"/>
 		</joint>
+		<transmission name="trans_${name}">
+				<type>transmission_interface/SimpleTransmission</type>
+				<joint name="${name}">
+					<hardwareInterface>hardware_interface/EffortJointInterface</hardwareInterface>
+				</joint>
+				<actuator name="motor_${name}">
+					<hardwareInterface>hardware_interface/EffortJointInterface</hardwareInterface>
+					<mechanicalReduction>1</mechanicalReduction>
+				</actuator>
+			</transmission>
     	</macro>
 </robot>
